Commit message: feat: added a 3d lidar sensor instead of a laser profiler, used the same meshes as microepsilon and  added a gitignore

File: kuka_trials/urdf/kr10r1420_macro.xacro (robot description, xacro)
@@ -17,4 +17,9 @@
         </geometry>
       </collision>
+      <inertial>
+        <origin xyz="0 0 0" rpy="0 0 0"/>
+        <mass value="10.0"/>
+        <inertia ixx="0.1" ixy="0.0" ixz="0.0" iyy="0.1" iyz="0.0" izz="0.1"/>
+      </inertial>
     </link>
     <link name="${prefix}link_1">
@@ -32,4 +37,9 @@
         </geometry>
       </collision>
+      <inertial>
+        <origin xyz="0 0 0" rpy="0 0 0"/>
+        <mass value="1.0"/>
+        <inertia ixx="0.1" ixy="0.0" ixz="0.0" iyy="0.1" iyz="0.0" izz="0.1"/>
+      </inertial>
     </link>
     <link name="${prefix}link_2">
@@ -47,4 +57,9 @@
         </geometry>
       </collision>
+      <inertial>
+        <origin xyz="0 0 0" rpy="0 0 0"/>
+        <mass value="1.0"/>
+        <inertia ixx="0.1" ixy="0.0" ixz="0.0" iyy="0.1" iyz="0.0" izz="0.1"/>
+      </inertial>
     </link>
     <link name="${prefix}link_3">
@@ -62,4 +77,9 @@
         </geometry>
       </collision>
+      <inertial>
+        <origin xyz="0 0 0" rpy="0 0 0"/>
+        <mass value="1.0"/>
+        <inertia ixx="0.1" ixy="0.0" ixz="0.0" iyy="0.1" iyz="0.0" izz="0.1"/>
+      </inertial>
     </link>
     <link name="${prefix}link_4">
@@ -77,4 +97,9 @@
         </geometry>
       </collision>
+      <inertial>
+        <origin xyz="0 0 0" rpy="0 0 0"/>
+        <mass value="1.0"/>
+        <inertia ixx="0.1" ixy="0.0" ixz="0.0" iyy="0.1" iyz="0.0" izz="0.1"/>
+      </inertial>
     </link>
     <link name="${prefix}link_5">
@@ -92,4 +117,9 @@
         </geometry>
       </collision>
+      <inertial>
+        <origin xyz="0 0 0" rpy="0 0 0"/>
+        <mass value="1.0"/>
+        <inertia ixx="0.1" ixy="0.0" ixz="0.0" iyy="0.1" iyz="0.0" izz="0.1"/>
+      </inertial>
     </link>
     <link name="${prefix}link_6">
@@ -107,7 +137,18 @@
         </geometry>
       </collision>
+      <inertial>
+        <origin xyz="0 0 0" rpy="0 0 0"/>
+        <mass value="1.0"/>
+        <inertia ixx="0.1" ixy="0.0" ixz="0.0" iyy="0.1" iyz="0.0" izz="0.1"/>
+      </inertial>
     </link>
     <!-- Following REP199, this frame shall be use to attach EEF or other equipment -->
-    <link name="${prefix}flange" />
+    <link name="${prefix}flange">
+      <inertial>
+        <origin xyz="0 0 0" rpy="0 0 0"/>
+        <mass value="0.1"/>
+        <inertia ixx="1e-4" ixy="0.0" ixz="0.0" iyy="1e-4" iyz="0.0" izz="1e-4"/>
+      </inertial>
+    </link>
     <joint name="${prefix}joint_a1" type="revolute">
       <origin xyz="0 0 0.450" rpy="0 0 0"/>

File: kuka_trials/urdf/robot.xacro (robot description, xacro)
@@ -2,4 +2,6 @@
 <robot name="kuka_kr10r1420" xmlns:xacro="http://wiki.ros.org/xacro">
   <xacro:include filename="kr10r1420_macro.xacro" />
+  <xacro:include filename="scancontrol_26x0_29x0_25_macro.xacro"/>
+  <xacro:microepsilon_scancontrol_26x0_29x0_25 prefix=""/>
   <xacro:kuka_kr10r1420 prefix=""/>
   <xacro:include filename="lidar.xacro" />

Commit message: chore: uploaded the kuka_config package and edited the robots urdf files

File: kuka_trials/urdf/kr10r1420_macro.xacro (robot description, xacro)
@@ -18,7 +18,7 @@
       </collision>
       <inertial>
-        <origin xyz="0 0 0" rpy="0 0 0"/>
-        <mass value="10.0"/>
-        <inertia ixx="0.1" ixy="0.0" ixz="0.0" iyy="0.1" iyz="0.0" izz="0.1"/>
+        <origin xyz="0 0 0" rpy="0 0 0" />
+        <mass value="320.0"/>
+        <inertia ixx="10.0" ixy="0.0" ixz="0.0" iyy="12.0" iyz="0.0" izz="5.0"/>
       </inertial>
     </link>
@@ -39,6 +39,6 @@
       <inertial>
         <origin xyz="0 0 0" rpy="0 0 0"/>
-        <mass value="1.0"/>
-        <inertia ixx="0.1" ixy="0.0" ixz="0.0" iyy="0.1" iyz="0.0" izz="0.1"/>
+        <mass value="20.0"/>
+        <inertia ixx="1.0" ixy="0.0" ixz="0.0" iyy="1.2" iyz="0.0" izz="0.8"/>
       </inertial>
     </link>
@@ -58,7 +58,7 @@
       </collision>
       <inertial>
-        <origin xyz="0 0 0" rpy="0 0 0"/>
-        <mass value="1.0"/>
-        <inertia ixx="0.1" ixy="0.0" ixz="0.0" iyy="0.1" iyz="0.0" izz="0.1"/>
+        <origin xyz="0 0 0" rpy="0 0 0" />
+        <mass value="18.0"/>
+        <inertia ixx="0.62" ixy="0.0" ixz="0.0" iyy="0.54" iyz="0.0" izz="0.35"/>
       </inertial>
     </link>
@@ -79,6 +79,6 @@
       <inertial>
         <origin xyz="0 0 0" rpy="0 0 0"/>
-        <mass value="1.0"/>
-        <inertia ixx="0.1" ixy="0.0" ixz="0.0" iyy="0.1" iyz="0.0" izz="0.1"/>
+        <mass value="15.0"/>
+        <inertia ixx="0.40" ixy="0.0" ixz="0.0" iyy="0.35" iyz="0.0" izz="0.25"/>
       </inertial>
     </link>
@@ -99,6 +99,6 @@
       <inertial>
         <origin xyz="0 0 0" rpy="0 0 0"/>
-        <mass value="1.0"/>
-        <inertia ixx="0.1" ixy="0.0" ixz="0.0" iyy="0.1" iyz="0.0" izz="0.1"/>
+        <mass value="9.0"/>
+        <inertia ixx="0.18" ixy="0.0" ixz="0.0" iyy="0.16" iyz="0.0" izz="0.10"/>
       </inertial>
     </link>
@@ -119,6 +119,6 @@
       <inertial>
         <origin xyz="0 0 0" rpy="0 0 0"/>
-        <mass value="1.0"/>
-        <inertia ixx="0.1" ixy="0.0" ixz="0.0" iyy="0.1" iyz="0.0" izz="0.1"/>
+        <mass value="6.0"/>
+        <inertia ixx="0.065" ixy="0.0" ixz="0.0" iyy="0.060" iyz="0.0" izz="0.040"/>
       </inertial>
     </link>
@@ -139,6 +139,6 @@
       <inertial>
         <origin xyz="0 0 0" rpy="0 0 0"/>
-        <mass value="1.0"/>
-        <inertia ixx="0.1" ixy="0.0" ixz="0.0" iyy="0.1" iyz="0.0" izz="0.1"/>
+        <mass value="4.0"/>
+        <inertia ixx="0.030" ixy="0.0" ixz="0.0" iyy="0.028" iyz="0.0" izz="0.020"/>
       </inertial>
     </link>
@@ -147,6 +147,6 @@
       <inertial>
         <origin xyz="0 0 0" rpy="0 0 0"/>
-        <mass value="0.1"/>
-        <inertia ixx="1e-4" ixy="0.0" ixz="0.0" iyy="1e-4" iyz="0.0" izz="1e-4"/>
+        <mass value="0.80"/>
+        <inertia ixx="0.0006" ixy="0.0" ixz="0.0" iyy="0.0006" iyz="0.0" izz="0.0008"/>
       </inertial>
     </link>
@@ -156,5 +156,5 @@
       <child link="${prefix}link_1"/>
       <axis xyz="0 0 -1"/>
-      <limit effort="0" lower="${radians(-170)}" upper="${radians(170)}" velocity="${radians(220)}"/>
+      <limit effort="500" lower="${radians(-170)}" upper="${radians(170)}" velocity="${radians(220)}"/>
     </joint>
     <joint name="${prefix}joint_a2" type="revolute">
@@ -163,5 +163,5 @@
       <child link="${prefix}link_2"/>
       <axis xyz="0 1 0"/>
-      <limit effort="0" lower="${radians(-185)}" upper="${radians(65)}" velocity="${radians(210)}"/>
+      <limit effort="500" lower="${radians(-185)}" upper="${radians(65)}" velocity="${radians(210)}"/>
     </joint>
     <joint name="${prefix}joint_a3" type="revolute">
@@ -170,5 +170,5 @@
       <child link="${prefix}link_3"/>
       <axis xyz="0 1 0"/>
-      <limit effort="0" lower="${radians(-137)}" upper="${radians(163)}" velocity="${radians(270)}"/>
+      <limit effort="500" lower="${radians(-137)}" upper="${radians(163)}" velocity="${radians(270)}"/>
     </joint>
     <joint name="${prefix}joint_a4" type="revolute">
@@ -177,5 +177,5 @@
       <child link="${prefix}link_4"/>
       <axis xyz="-1 0 0"/>
-      <limit effort="0" lower="${radians(-185)}" upper="${radians(185)}" velocity="${radians(381)}"/>
+      <limit effort="500" lower="${radians(-185)}" upper="${radians(185)}" velocity="${radians(381)}"/>
     </joint>
     <joint name="${prefix}joint_a5" type="revolute">
@@ -184,5 +184,5 @@
       <child link="${prefix}link_5"/>
       <axis xyz="0 1 0"/>
-      <limit effort="0" lower="${radians(-120)}" upper="${radians(120)}" velocity="${radians(311)}"/>
+      <limit effort="500" lower="${radians(-120)}" upper="${radians(120)}" velocity="${radians(311)}"/>
     </joint>
     <joint name="${prefix}joint_a6" type="revolute">
@@ -191,5 +191,5 @@
       <child link="${prefix}link_6"/>
       <axis xyz="-1 0 0"/>
-      <limit effort="0" lower="${radians(-350)}" upper="${radians(350)}" velocity="${radians(492)}"/>
+      <limit effort="500" lower="${radians(-350)}" upper="${radians(350)}" velocity="${radians(492)}"/>
     </joint>
     <joint name="${prefix}joint_a6-flange" type="fixed">
@@ -198,18 +198,4 @@
       <origin xyz="0 0 0" rpy="0 0 0"/>
     </joint>
-    <!-- ROS base_link to KUKA $ROBROOT coordinate system transform -->
-    <link name="${prefix}base" />
-    <joint name="${prefix}base_link-base" type="fixed">
-      <origin xyz="0 0 0" rpy="0 0 0"/>
-      <parent link="${prefix}base_link"/>
-      <child link="${prefix}base"/>
-    </joint>
-    <!-- This frame corresponds to the $TOOL coordinate system in KUKA KRC controllers -->
-    <link name="${prefix}tool0" />
-    <joint name="${prefix}flange-tool0" type="fixed">
-      <parent link="${prefix}flange"/>
-      <child link="${prefix}tool0"/>
-      <origin xyz="0 0 0" rpy="0 ${radians(90)} 0"/>
-    </joint>
   </xacro:macro>
 </robot>

File: kuka_trials/urdf/lidar.xacro (robot description, xacro)
@@ -2,7 +2,29 @@
 <robot name="kuka_kr10r1420"
     xmlns:xacro="http://wiki.ros.org/xacro">
+    <link name="lidar_link">
+        <visual>
+            <origin xyz="0 0 0" rpy="${pi/2} 0 ${pi/2}"/>
+            <geometry>
+                <mesh filename="package://kuka_trials/meshes/visual.dae"/>
+            </geometry>
+            <material name="microepsilon_silver">
+                <color rgba="0.7 0.7 0.7 1.0"/>
+            </material>
+        </visual>
+        <collision>
+            <origin xyz="0 0 0" rpy="${pi/2} 0 ${pi/2}"/>
+            <geometry>
+                <mesh filename="package://kuka_trials/meshes/collision.stl"/>
+            </geometry>
+        </collision>
+        <inertial>
+            <origin xyz="0 0 0" rpy="0 0 0"/>
+            <mass value="0.1"/>
+            <inertia ixx="0.1" ixy="0.0" ixz="0.0" iyy="0.1" iyz="0.0" izz="0.1"/>
+        </inertial>
+    </link>
     <joint name="flange_to_lidar" type="fixed">
         <parent link="flange"/>
-        <child link="microepsilon"/>
+        <child link="lidar_link"/>
         <origin xyz="0.05 0 0" rpy="0 0 0"/>
     </joint>
@@ -12,5 +34,5 @@
         </plugin>
     </gazebo>
-    <gazebo reference="microepsilon">
+    <gazebo reference="lidar_link">
         <sensor name="gpu_lidar" type="gpu_lidar">
             <visualize>true</visualize>
@@ -18,5 +40,5 @@
             <update_rate>5</update_rate>
             <topic>scan</topic>
-            <gz_frame_id>microepsilon</gz_frame_id>
+            <gz_frame_id>lidar_link</gz_frame_id>
             <lidar>
                 <scan>

File: kuka_trials/urdf/robot.xacro (robot description, xacro)
@@ -2,6 +2,4 @@
 <robot name="kuka_kr10r1420" xmlns:xacro="http://wiki.ros.org/xacro">
   <xacro:include filename="kr10r1420_macro.xacro" />
-  <xacro:include filename="scancontrol_26x0_29x0_25_macro.xacro"/>
-  <xacro:microepsilon_scancontrol_26x0_29x0_25 prefix=""/>
   <xacro:kuka_kr10r1420 prefix=""/>
   <xacro:include filename="lidar.xacro" />
