Commit message: chore: moved joint from robot.xacro to drill_bit.urdf.xacro and edited the gazebo launch file to bridge topics from gz to ros

File: kuka_trials/urdf/drill_bit.urdf.xacro (robot description, xacro)
@@ -44,3 +44,8 @@
     <limit effort="10.0" velocity="1.0" lower="-3.14" upper="3.14"/>
   </joint>
+  <joint name="robot_to_drill_bit" type="fixed">
+    <parent link="base_link"/>
+    <child link="cylinder_link"/>
+    <origin xyz="2 0 0" rpy="0 0 0"/>
+  </joint>
 </robot>

File: kuka_trials/urdf/robot.xacro (robot description, xacro)
@@ -5,8 +5,3 @@
   <xacro:include filename="lidar.xacro" />
   <xacro:include filename="drill_bit.urdf.xacro"/>
-  <joint name="robot_to_drill_bit" type="fixed">
-    <parent link="base_link"/>
-    <child link="cylinder_link"/>
-    <origin xyz="2 0 0" rpy="0 0 0"/>
-  </joint>
 </robot>

Commit message: fixed pointcloud scan demo

File: kuka_trials/urdf/drill_bit.urdf.xacro (robot description, xacro)
@@ -42,5 +42,5 @@
     <origin xyz="0 0 0.5" rpy="0 0 0"/>
     <axis xyz="0 0 1"/>
-    <limit effort="10.0" velocity="1.0" lower="-3.14" upper="3.14"/>
+    <limit effort="10.0" velocity="1.0" lower="0" upper="6.28"/>
   </joint>
   <joint name="robot_to_drill_bit" type="fixed">

File: kuka_trials/urdf/lidar.xacro (robot description, xacro)
@@ -52,6 +52,6 @@
                         <samples>640</samples>
                         <resolution>1</resolution>
-                        <min_angle>0.3735004599267865</min_angle>
-                        <max_angle>0.4363323129985824</max_angle>
+                        <min_angle>-0.1867</min_angle>
+                        <max_angle>-0.1867</max_angle>
                     </vertical>
                 </scan>

Commit message: feat: removed the rotary table and fixated the drill bit in an inverted manner

File: kuka_trials/urdf/drill_bit.urdf.xacro (robot description, xacro)
@@ -1,23 +1,9 @@
 <?xml version="1.0" encoding="UTF-8"?>
 <robot name="drill_bit_module">
-  <link name="cylinder_link">
-    <visual>
-      <geometry>
-        <cylinder radius="0.4" length="0.2"/>
-      </geometry>
-      <origin xyz="0 0 0.1" rpy="0 0 0"/>
-    </visual>
-    <collision>
-      <geometry>
-        <cylinder radius="0.4" length="0.2"/>
-      </geometry>
-      <origin xyz="0 0 0.1" rpy="0 0 0"/>
-    </collision>
-  </link>
   <link name="drill_bit">
     <visual>
       <origin xyz="0 0 0" rpy="0 0 0"/>
       <geometry>
-        <mesh filename="package://kuka_trials/meshes/Bit.dae" scale="2 2 2"/>
+        <mesh filename="package://kuka_trials/meshes/Bit.dae" scale="1.5 1.5 1.5"/>
       </geometry>
         <material name="Red">
@@ -28,5 +14,5 @@
       <origin xyz="0 0 0" rpy="0 0 0"/>
       <geometry>
-        <mesh filename="package://kuka_trials/meshes/Bit.dae" scale="2 2 2"/>
+        <mesh filename="package://kuka_trials/meshes/Bit.dae" scale="1.5 1.5 1.5"/>
       </geometry>
     </collision>
@@ -37,14 +23,8 @@
     </inertial>
   </link>
-  <joint name="cylinder_to_drill_bit" type="continuous">
-    <parent link="cylinder_link"/>
-    <child link="drill_bit"/>
-    <origin xyz="0 0 0.5" rpy="0 0 0"/>
-    <axis xyz="0 0 1"/>
-  </joint>
   <joint name="robot_to_drill_bit" type="fixed">
     <parent link="base_link"/>
-    <child link="cylinder_link"/>
-    <origin xyz="2 0 0" rpy="0 0 0"/>
+    <child link="drill_bit"/>
+    <origin xyz="0.0 0 1.625" rpy="3.14159 0 0"/>
   </joint>
 </robot>
