Commit message: added the rotary table and drill bit to moveit

File: kuka_config/config/kuka_kr10r1420.ros2_control.xacro (robot description, xacro)
@@ -49,4 +49,9 @@
         <state_interface name="velocity"/>
       </joint>
+      <joint name="cylinder_to_drill_bit">
+        <command_interface name="position"/>
+        <state_interface name="position"/>
+        <state_interface name="velocity"/>
+      </joint>
     </ros2_control>
     <gazebo>

File: kuka_trials/urdf/robot.xacro (robot description, xacro)
@@ -4,3 +4,9 @@
   <xacro:kuka_kr10r1420 prefix=""/>
   <xacro:include filename="lidar.xacro" />
+  <xacro:include filename="drill_bit.urdf.xacro"/>
+  <joint name="robot_to_drill_bit" type="fixed">
+    <parent link="base_link"/>
+    <child link="cylinder_link"/>
+    <origin xyz="2 0 0" rpy="0 0 0"/>
+  </joint>
 </robot>

Commit message: feat: used a velocity controller instead of a joint trajectory controller for the rotary table

File: kuka_config/config/kuka_kr10r1420.ros2_control.xacro (robot description, xacro)
@@ -5,5 +5,5 @@
     <ros2_control name="${name}" type="system">
       <hardware>
-        <plugin>ign_ros2_control/IgnitionSystem</plugin>
+        <plugin>gz_ros2_control/GazeboSimSystem</plugin>
       </hardware>
       <joint name="joint_a1">
@@ -50,5 +50,5 @@
       </joint>
       <joint name="cylinder_to_drill_bit">
-        <command_interface name="position"/>
+        <command_interface name="velocity"/>
         <state_interface name="position"/>
         <state_interface name="velocity"/>

File: kuka_trials/urdf/drill_bit.urdf.xacro (robot description, xacro)
@@ -37,10 +37,9 @@
     </inertial>
   </link>
-  <joint name="cylinder_to_drill_bit" type="revolute">
+  <joint name="cylinder_to_drill_bit" type="continuous">
     <parent link="cylinder_link"/>
     <child link="drill_bit"/>
     <origin xyz="0 0 0.5" rpy="0 0 0"/>
     <axis xyz="0 0 1"/>
-    <limit effort="10.0" velocity="1.0" lower="-3.14" upper="3.14"/>
   </joint>
   <joint name="robot_to_drill_bit" type="fixed">
