Commit message: Add laser profiler URDF/Xacro and integrate into robot model

File: kuka_kr10_r1440/urdf/my_robot.urdf.xacro (robot description, xacro)
@@ -2,3 +2,9 @@
 <robot name="my_robot" xmlns:xacro="http://www.ros.org/wiki/xacro">
     <xacro:include filename="kuka_kr10_r1440.xacro"/>
+    <xacro:include filename="laser_profiler.xacro"/>
+    <joint name="laser_profiler_base_joint" type="fixed">
+        <parent link="tool_link"/>
+        <child link="lp_link"/>
+        <origin xyz="0 0 0" rpy="0 0 0"/>
+    </joint>
 </robot>
