Commit message: feat: update URDF structure by renaming and adding new robot model, including tool link and joint definitions

File: kuka_kr10_r1440/urdf/kuka_kr10_r1440.xacro (robot description, xacro)
@@ -392,3 +392,9 @@
       velocity="8.238" />
   </joint>
+  <link name="tool_link" />
+  <joint name="hand_tool_joint" type="fixed">
+    <parent link="tip"/>
+    <child link="tool_link"/>
+    <origin xyz="0.03 0 0" rpy="0 0 0"/>
+  </joint>
 </robot>

Commit message: Refactor package name from 'kuka_kr10_r1440' to 'my_robot_description'

File: kuka_kr10_r1440/urdf/kuka_kr10_r1440.xacro (robot description, xacro)
@@ -26,19 +26,19 @@
       <geometry>
         <mesh
-          filename="package://kuka_kr10_r1440/meshes/base_link.STL" />
-      </geometry>
-      <material
-        name="">
-        <color
-          rgba="0.792156862745098 0.819607843137255 0.933333333333333 1" />
-      </material>
-    </visual>
-    <collision>
-      <origin
-        xyz="0 0 0"
-        rpy="0 0 0" />
-      <geometry>
-        <mesh
-          filename="package://kuka_kr10_r1440/meshes/base_link.STL" />
+          filename="package://my_robot_description/meshes/base_link.STL" />
+      </geometry>
+      <material
+        name="">
+        <color
+          rgba="0.792156862745098 0.819607843137255 0.933333333333333 1" />
+      </material>
+    </visual>
+    <collision>
+      <origin
+        xyz="0 0 0"
+        rpy="0 0 0" />
+      <geometry>
+        <mesh
+          filename="package://my_robot_description/meshes/base_link.STL" />
       </geometry>
     </collision>
@@ -66,19 +66,19 @@
       <geometry>
         <mesh
-          filename="package://kuka_kr10_r1440/meshes/main.STL" />
-      </geometry>
-      <material
-        name="">
-        <color
-          rgba="0.792156862745098 0.819607843137255 0.933333333333333 1" />
-      </material>
-    </visual>
-    <collision>
-      <origin
-        xyz="0 0 0"
-        rpy="0 0 0" />
-      <geometry>
-        <mesh
-          filename="package://kuka_kr10_r1440/meshes/main.STL" />
+          filename="package://my_robot_description/meshes/main.STL" />
+      </geometry>
+      <material
+        name="">
+        <color
+          rgba="0.792156862745098 0.819607843137255 0.933333333333333 1" />
+      </material>
+    </visual>
+    <collision>
+      <origin
+        xyz="0 0 0"
+        rpy="0 0 0" />
+      <geometry>
+        <mesh
+          filename="package://my_robot_description/meshes/main.STL" />
       </geometry>
     </collision>
@@ -124,19 +124,19 @@
       <geometry>
         <mesh
-          filename="package://kuka_kr10_r1440/meshes/shoulder.STL" />
-      </geometry>
-      <material
-        name="">
-        <color
-          rgba="0.792156862745098 0.819607843137255 0.933333333333333 1" />
-      </material>
-    </visual>
-    <collision>
-      <origin
-        xyz="0 0 0"
-        rpy="0 0 0" />
-      <geometry>
-        <mesh
-          filename="package://kuka_kr10_r1440/meshes/shoulder.STL" />
+          filename="package://my_robot_description/meshes/shoulder.STL" />
+      </geometry>
+      <material
+        name="">
+        <color
+          rgba="0.792156862745098 0.819607843137255 0.933333333333333 1" />
+      </material>
+    </visual>
+    <collision>
+      <origin
+        xyz="0 0 0"
+        rpy="0 0 0" />
+      <geometry>
+        <mesh
+          filename="package://my_robot_description/meshes/shoulder.STL" />
       </geometry>
     </collision>
@@ -182,19 +182,19 @@
       <geometry>
         <mesh
-          filename="package://kuka_kr10_r1440/meshes/elbow.STL" />
-      </geometry>
-      <material
-        name="">
-        <color
-          rgba="0.792156862745098 0.819607843137255 0.933333333333333 1" />
-      </material>
-    </visual>
-    <collision>
-      <origin
-        xyz="0 0 0"
-        rpy="0 0 0" />
-      <geometry>
-        <mesh
-          filename="package://kuka_kr10_r1440/meshes/elbow.STL" />
+          filename="package://my_robot_description/meshes/elbow.STL" />
+      </geometry>
+      <material
+        name="">
+        <color
+          rgba="0.792156862745098 0.819607843137255 0.933333333333333 1" />
+      </material>
+    </visual>
+    <collision>
+      <origin
+        xyz="0 0 0"
+        rpy="0 0 0" />
+      <geometry>
+        <mesh
+          filename="package://my_robot_description/meshes/elbow.STL" />
       </geometry>
     </collision>
@@ -240,19 +240,19 @@
       <geometry>
         <mesh
-          filename="package://kuka_kr10_r1440/meshes/forearm.STL" />
-      </geometry>
-      <material
-        name="">
-        <color
-          rgba="0.792156862745098 0.819607843137255 0.933333333333333 1" />
-      </material>
-    </visual>
-    <collision>
-      <origin
-        xyz="0 0 0"
-        rpy="0 0 0" />
-      <geometry>
-        <mesh
-          filename="package://kuka_kr10_r1440/meshes/forearm.STL" />
+          filename="package://my_robot_description/meshes/forearm.STL" />
+      </geometry>
+      <material
+        name="">
+        <color
+          rgba="0.792156862745098 0.819607843137255 0.933333333333333 1" />
+      </material>
+    </visual>
+    <collision>
+      <origin
+        xyz="0 0 0"
+        rpy="0 0 0" />
+      <geometry>
+        <mesh
+          filename="package://my_robot_description/meshes/forearm.STL" />
       </geometry>
     </collision>
@@ -298,19 +298,19 @@
       <geometry>
         <mesh
-          filename="package://kuka_kr10_r1440/meshes/end_effector.STL" />
-      </geometry>
-      <material
-        name="">
-        <color
-          rgba="0.792156862745098 0.819607843137255 0.933333333333333 1" />
-      </material>
-    </visual>
-    <collision>
-      <origin
-        xyz="0 0 0"
-        rpy="0 0 0" />
-      <geometry>
-        <mesh
-          filename="package://kuka_kr10_r1440/meshes/end_effector.STL" />
+          filename="package://my_robot_description/meshes/end_effector.STL" />
+      </geometry>
+      <material
+        name="">
+        <color
+          rgba="0.792156862745098 0.819607843137255 0.933333333333333 1" />
+      </material>
+    </visual>
+    <collision>
+      <origin
+        xyz="0 0 0"
+        rpy="0 0 0" />
+      <geometry>
+        <mesh
+          filename="package://my_robot_description/meshes/end_effector.STL" />
       </geometry>
     </collision>
@@ -356,19 +356,19 @@
       <geometry>
         <mesh
-          filename="package://kuka_kr10_r1440/meshes/tip.STL" />
-      </geometry>
-      <material
-        name="">
-        <color
-          rgba="0.792156862745098 0.819607843137255 0.933333333333333 1" />
-      </material>
-    </visual>
-    <collision>
-      <origin
-        xyz="0 0 0"
-        rpy="0 0 0" />
-      <geometry>
-        <mesh
-          filename="package://kuka_kr10_r1440/meshes/tip.STL" />
+          filename="package://my_robot_description/meshes/tip.STL" />
+      </geometry>
+      <material
+        name="">
+        <color
+          rgba="0.792156862745098 0.819607843137255 0.933333333333333 1" />
+      </material>
+    </visual>
+    <collision>
+      <origin
+        xyz="0 0 0"
+        rpy="0 0 0" />
+      <geometry>
+        <mesh
+          filename="package://my_robot_description/meshes/tip.STL" />
       </geometry>
     </collision>

File: kuka_kr10_r1440/urdf/laser_profiler.xacro (robot description, xacro)
@@ -6,5 +6,5 @@
             <origin xyz="0.05 0 0" rpy="0 0 ${pi/2}"/>
             <geometry>
-                <mesh filename="package://kuka_kr10_r1440/meshes/scanControl_laser_profiler/laser_profiler_visual.dae"/>
+                <mesh filename="package://my_robot_description/meshes/scanControl_laser_profiler/laser_profiler_visual.dae"/>
             </geometry>
             <material name="microepsilon_silver">
@@ -15,5 +15,5 @@
             <origin xyz="0.05 0 0" rpy="0 0 0"/>
             <geometry>
-                <mesh filename="package://kuka_kr10_r1440/meshes/scanControl_laser_profiler/laser_profiler_collision.stl"/>
+                <mesh filename="package://my_robot_description/meshes/scanControl_laser_profiler/laser_profiler_collision.stl"/>
             </geometry>
         </collision>
