Commit message: Add drill bit mesh and XACRO file to robot description

File: my_robot_description/urdf/my_robot.urdf.xacro (robot description, xacro)
@@ -3,4 +3,5 @@
     <xacro:include filename="kuka_kr10_r1440.xacro"/>
     <xacro:include filename="laser_profiler.xacro"/>
+    <xacro:include filename="drill_bit.xacro" />
     <joint name="laser_profiler_base_joint" type="fixed">
         <parent link="tool_link"/>
@@ -8,3 +9,8 @@
         <origin xyz="0 0 0" rpy="0 0 0"/>
     </joint>
+    <joint name="robot_to_drill_bit" type="fixed">
+        <parent link="base_link"/>
+        <child link="drill_bit"/>
+        <origin xyz="0.0 0 1.625" rpy="3.14159 0 0"/>
+  </joint>
 </robot>
